Commit message: fix joint limits

File: vesc_hw_interface/launch/test.xacro (robot description, xacro)
@@ -1,5 +1,5 @@
 <?xml version="1.0"?>
 <robot name="vesc_test">
-  <link name="base_link"></link>
+  <link name="base_link"/>
   <joint name="arm_joint" type="revolute">
     <parent link="base_link"/>
@@ -7,6 +7,6 @@
     <origin xyz="0 0 0" rpy="0 0 0"/>
     <axis xyz="0 0 1"/>
-    <limit effort="100" lower="100" upper="100" velocity="100"/>
+    <limit effort="100" lower="-100" upper="100" velocity="100"/>
   </joint>
-  <link name="arm_link"></link>
+  <link name="arm_link"/>
 </robot>

Commit message: rename to vesc_*

File: vesc_hw_interface/launch/test.xacro (robot description, xacro)
@@ -2,11 +2,11 @@
 <robot name="vesc_test">
   <link name="base_link"/>
-  <joint name="arm_joint" type="revolute">
+  <joint name="vesc_joint" type="revolute">
     <parent link="base_link"/>
-    <child link="arm_link"/>
+    <child link="vesc_link"/>
     <origin xyz="0 0 0" rpy="0 0 0"/>
     <axis xyz="0 0 1"/>
     <limit effort="100" lower="-100" upper="100" velocity="100"/>
   </joint>
-  <link name="arm_link"/>
+  <link name="vesc_link"/>
 </robot>

Commit message: Fix enforceLimits(period)

File: vesc_hw_interface/launch/test.xacro (robot description, xacro)
@@ -7,5 +7,6 @@
     <origin xyz="0 0 0" rpy="0 0 0"/>
     <axis xyz="0 0 1"/>
-    <limit effort="100" lower="-100" upper="100" velocity="100"/>
+    <limit effort="100" lower="-100" upper="100" velocity="1000"/>
+    <safety_controller k_velocity="10" k_position="15" soft_lower_limit="-2.0" soft_upper_limit="0.5" />
   </joint>
   <link name="vesc_link"/>
