Commit message: fix samples

File: vesc_hw_interface/launch/position_duty_test.ros2_control.xacro (robot description, xacro)
@@ -1,4 +1,13 @@
 <?xml version="1.0" encoding="UTF-8"?>
 <robot xmlns:xacro="http://www.ros.org/wiki/xacro">
+  <link name="base_link"/>
+  <link name="vesc_link"/>
+  <joint name="vesc_joint" type="prismatic">
+    <parent link="base_link"/>
+    <child link="vesc_link"/>
+    <origin xyz="0 0 0" rpy="0 0 0"/>
+    <axis xyz="0 0 1"/>
+    <limit lower="-1.0" upper="1.0" velocity="10" effort="5000"/>
+  </joint>
   <ros2_control name="vesc" type="actuator">
     <hardware>
@@ -31,5 +40,5 @@
       <param name="servo/endstop_threshold">0.8</param>
       <param name="servo/endstop_margin">0.02</param>
-      <param name="command_mode">position</param>
+      <param name="command_mode">position_duty</param>
     </hardware>
     <joint name="vesc_joint">

File: vesc_hw_interface/launch/velocity_duty_test.ros2_control.xacro (robot description, xacro)
@@ -1,8 +1,17 @@
 <?xml version="1.0" encoding="UTF-8"?>
 <robot xmlns:xacro="http://www.ros.org/wiki/xacro">
+  <link name="base_link"/>
+  <link name="vesc_link"/>
+  <joint name="vesc_joint" type="continuous">
+    <parent link="base_link"/>
+    <child link="vesc_link"/>
+    <origin xyz="0 0 0" rpy="0 0 0"/>
+    <axis xyz="0 0 1"/>
+    <limit lower="-1.0" upper="1.0" velocity="10" effort="5000"/>
+  </joint>
   <ros2_control name="vesc" type="actuator">
     <hardware>
       <plugin>vesc_hw_interface/VescHwInterface</plugin>
-      <param name="port">/dev/ttyVESC_left</param>
+      <param name="port">/dev/ttyACM0</param>
       <param name="gear_ratio">0.230769</param>
       <param name="torque_const">1.0</param>

Commit message: added new samples

File: vesc_hw_interface/launch/position_duty_test.ros2_control.xacro (robot description, xacro)
@@ -1,4 +1,4 @@
 <?xml version="1.0" encoding="UTF-8"?>
-<robot xmlns:xacro="http://www.ros.org/wiki/xacro">
+<robot xmlns:xacro="http://www.ros.org/wiki/xacro" name="test">
   <link name="base_link"/>
   <link name="vesc_link"/>

File: vesc_hw_interface/launch/position_test.ros2_control.xacro (robot description, xacro)
@@ -3,5 +3,5 @@
   <link name="base_link"/>
   <link name="vesc_link"/>
-  <joint name="vesc_joint" type="continuous">
+  <joint name="vesc_joint" type="prismatic">
     <parent link="base_link"/>
     <child link="vesc_link"/>
@@ -14,20 +14,6 @@
       <plugin>vesc_hw_interface/VescHwInterface</plugin>
       <param name="port">/dev/ttyACM0</param>
-      <param name="gear_ratio">0.230769</param>
-      <param name="torque_const">1.0</param>
-      <param name="num_hall_sensors">3</param>
-      <param name="screw_lead">1.0</param>
-      <param name="num_rotor_poles">20</param>
-      <param name="motor/Kp">0.1</param>
-      <param name="motor/Ki">0.01</param>
-      <param name="motor/Kd">0.02</param>
-      <param name="motor/i_clamp">1.0</param>
-      <param name="motor/duty_limiter">1.0</param>
-      <param name="motor/antiwindup">true</param>
-      <param name="motor/control_rate">100.0</param>
-      <param name="motor/enable_smooth_diff">true</param>
-      <param name="motor/smooth_diff/max_sample_sec">0.2</param>
-      <param name="motor/smooth_diff/max_smooth_step">10</param>
-      <param name="command_mode">velocity_duty</param>
+      <param name="servo/calibration">false</param>
+      <param name="command_mode">position</param>
     </hardware>
     <joint name="vesc_joint">

File: vesc_hw_interface/launch/velocity_test.ros2_control.xacro (robot description, xacro)
@@ -14,20 +14,5 @@
       <plugin>vesc_hw_interface/VescHwInterface</plugin>
       <param name="port">/dev/ttyACM0</param>
-      <param name="gear_ratio">0.230769</param>
-      <param name="torque_const">1.0</param>
-      <param name="num_hall_sensors">3</param>
-      <param name="screw_lead">1.0</param>
-      <param name="num_rotor_poles">20</param>
-      <param name="motor/Kp">0.1</param>
-      <param name="motor/Ki">0.01</param>
-      <param name="motor/Kd">0.02</param>
-      <param name="motor/i_clamp">1.0</param>
-      <param name="motor/duty_limiter">1.0</param>
-      <param name="motor/antiwindup">true</param>
-      <param name="motor/control_rate">100.0</param>
-      <param name="motor/enable_smooth_diff">true</param>
-      <param name="motor/smooth_diff/max_sample_sec">0.2</param>
-      <param name="motor/smooth_diff/max_smooth_step">10</param>
-      <param name="command_mode">velocity_duty</param>
+      <param name="command_mode">velocity</param>
     </hardware>
     <joint name="vesc_joint">
